File: pcb/2_assemble/jtnk66w.kicad_pcb (KiCad board)
At the start: 2 copper layers, 376.2 x 83.3 mm, 224 parts, among them J1 Conn_01x02, J10 Conn_01x01, J11 Conn_01x01, J12 Conn_01x01, J13 Conn_01x01, J14 Conn_01x01, J15 Conn_01x01, J16 Conn_01x01, J17 Conn_01x01, J18 Conn_01x01, J19 Conn_01x01, J2 Conn_01x01, J20 Conn_01x01, J21 Conn_01x01, J22 Conn_01x01, J23 Conn_01x01, J3 Conn_01x01, J4 Conn_01x01, J5 Conn_01x01, J6 Conn_01x01, J7 Conn_01x01, J8 Conn_01x01, J9 Conn_01x01, SW1 SW_PUSH, SW10 SW_PUSH, SW11 SW_PUSH, SW12 SW_PUSH, SW13 SW_PUSH, SW14 SW_PUSH, SW15 SW_PUSH, SW16 SW_PUSH, SW17 SW_PUSH, SW18 SW_PUSH, SW19 SW_PUSH, SW2 Rotary_Encoder_Switch, SW20 SW_PUSH, SW21 SW_PUSH, SW22 SW_PUSH, SW23 SW_PUSH, SW24 SW_PUSH, SW25 SW_PUSH, SW26 SW_PUSH, SW27 SW_PUSH, SW28 SW_PUSH, SW29 SW_PUSH, SW3 SW_PUSH, SW30 SW_PUSH, SW31 SW_PUSH, SW32 SW_PUSH, SW33 SW_PUSH, SW34 SW_PUSH, SW35 SW_PUSH, SW36 SW_PUSH, SW37 SW_PUSH, SW38 SW_PUSH, SW39 SW_PUSH, SW4 SW_PUSH, SW40 SW_PUSH, SW41 SW_PUSH, SW42 SW_PUSH, SW43 SW_PUSH, SW44 SW_PUSH, SW45 SW_PUSH, SW46 SW_PUSH, SW47 SW_PUSH, SW48 SW_PUSH, SW49 SW_PUSH, SW5 SW_PUSH, SW50 SW_PUSH, SW51 SW_PUSH, SW52 SW_PUSH, SW53 SW_PUSH, SW54 SW_PUSH, SW55 SW_PUSH, SW56 SW_PUSH, SW57 SW_PUSH, SW58 SW_PUSH, SW59 SW_PUSH, SW6 SW_PUSH, SW60 SW_PUSH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

Commit message: blender
Parts:
- added G***: LOGO, 2_assemble:logo, F.Cu at (198.8, 72.8)
- SW10, SW14, SW6: footprint kbd_SW:CherryMX_Hotswap_1u -> kbd_SW:CherryMX_Hotswap_1.25u
- SW18, SW25: footprint kbd_SW:CherryMX_Hotswap_1u -> kbd_SW:CherryMX_Hotswap_2u
- SW3, SW48: footprint kbd_SW:CherryMX_Hotswap_1u -> kbd_SW:CherryMX_Hotswap_1.5u
- SW4: footprint kbd_SW:CherryMX_Hotswap_1u -> kbd_SW:CherryMX_Hotswap_1.75u
- SW5, SW51: footprint kbd_SW:CherryMX_Hotswap_1u -> kbd_SW:CherryMX_Hotswap_2.25u
Connections:
- D56 pad 2: Net-(D56-Pad2) -> Row1
- D57 pad 2: Net-(D57-Pad2) -> Row2
- D60 pad 2: Net-(D56-Pad2) -> Row1
- D61 pad 2: Net-(D57-Pad2) -> Row2
- D64 pad 2: Net-(D56-Pad2) -> Row1
- D65 pad 2: Net-(D57-Pad2) -> Row2
- L1 pad 3: Net-(L1-Pad3) -> LED
Routing:
- net Col7: track 599.5 -> 521.3 mm, vias 11 -> 10
- net Col1: track 447.9 -> 378.4 mm, vias 13 -> 10
- net Net-(D57-Pad2): track 67.7 -> 0.00 mm
- net Col6: track 544.8 -> 494.5 mm, vias 15 -> 12
- net LED: track 0.00 -> 49.7 mm
- net Net-(D56-Pad2): track 47.2 -> 0.00 mm
- net Row3: track 487.3 -> 444.4 mm, vias 11 -> 4
- net GND: track 1844.1 -> 1802.2 mm
- net Row0: track 410.3 -> 451.0 mm, vias 2 -> 7
- net Row2: track 406.9 -> 440.1 mm, vias 7 -> 4
- net Col8: track 590.9 -> 559.2 mm, vias 6 -> 4
- net Row1: track 370.9 -> 394.1 mm, vias 5 -> 3
- net Net-(D55-Pad1): track 34.2 -> 12.4 mm
- net Net-(D66-Pad1): track 13.2 -> 34.1 mm, vias 2 -> 0
- net VCC: track 1608.3 -> 1588.1 mm
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Other:
- board text added: "jtnk66w rev.0991 tanakajunjun@gmail.com"
- board text removed: "jtnk66w rev.099 tanakajunjun@gmail.com"
