File: pcb/2_assemble/jtnk66w.sch (KiCad schematic (older format))
At the start: 218 parts, among them J1 Conn_01x02, J10 Conn_01x01, J11 Conn_01x01, J12 Conn_01x01, J13 Conn_01x01, J14 Conn_01x01, J15 Conn_01x01, J16 Conn_01x01, J17 Conn_01x01, J2 Conn_01x01, J3 Conn_01x01, J4 Conn_01x01, J5 Conn_01x01, J6 Conn_01x01, J7 Conn_01x01, J8 Conn_01x01, J9 Conn_01x01, SW1 SW_PUSH, SW10 SW_PUSH, SW11 SW_PUSH, SW12 SW_PUSH, SW13 SW_PUSH, SW14 SW_PUSH, SW15 SW_PUSH, SW16 SW_PUSH, SW17 SW_PUSH, SW18 SW_PUSH, SW19 SW_PUSH, SW2 Rotary_Encoder_Switch, SW20 SW_PUSH, SW21 SW_PUSH, SW22 SW_PUSH, SW23 SW_PUSH, SW24 SW_PUSH, SW25 SW_PUSH, SW26 SW_PUSH, SW27 SW_PUSH, SW28 SW_PUSH, SW29 SW_PUSH, SW3 SW_PUSH, SW30 SW_PUSH, SW31 SW_PUSH, SW32 SW_PUSH, SW33 SW_PUSH, SW34 SW_PUSH, SW35 SW_PUSH, SW36 SW_PUSH, SW37 SW_PUSH, SW38 SW_PUSH, SW39 SW_PUSH, SW4 SW_PUSH, SW40 SW_PUSH, SW41 SW_PUSH, SW42 SW_PUSH, SW43 SW_PUSH, SW44 SW_PUSH, SW45 SW_PUSH, SW46 SW_PUSH, SW47 SW_PUSH, SW48 SW_PUSH, SW49 SW_PUSH, SW5 SW_PUSH, SW50 SW_PUSH, SW51 SW_PUSH, SW52 SW_PUSH, SW53 SW_PUSH, SW54 SW_PUSH, SW55 SW_PUSH, SW56 SW_PUSH, SW57 SW_PUSH, SW58 SW_PUSH, SW59 SW_PUSH, SW6 SW_PUSH, SW60 SW_PUSH, SW61 SW_PUSH, SW62 SW_PUSH, SW63 SW_PUSH, SW64 SW_PUSH, SW65 SW_PUSH, SW66 SW_PUSH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

Commit message: blender
Parts:
- SW10, SW14, SW6: footprint kbd_SW:CherryMX_Hotswap_1u -> kbd_SW:CherryMX_Hotswap_1.25u
- SW18, SW25: footprint kbd_SW:CherryMX_Hotswap_1u -> kbd_SW:CherryMX_Hotswap_2u
- SW3, SW48: footprint kbd_SW:CherryMX_Hotswap_1u -> kbd_SW:CherryMX_Hotswap_1.5u
- SW4: footprint kbd_SW:CherryMX_Hotswap_1u -> kbd_SW:CherryMX_Hotswap_1.75u
- SW5, SW51: footprint kbd_SW:CherryMX_Hotswap_1u -> kbd_SW:CherryMX_Hotswap_2.25u
Connections:
- net LED: now also L1.3 (DIN)
- net Row1: now also D56.2 (A), D60.2 (A), D64.2 (A)
- net Row2: now also D57.2 (A), D61.2 (A), D65.2 (A)
Changed lines of the file:
@@
 F 0 "SW25" H 6050 6080 50  0000 C CNN
 F 1 "SW_PUSH" H 6050 5989 50  0000 C CNN
-F 2 "kbd_SW:CherryMX_Hotswap_1u" H 6050 5825 50  0001 C CNN
+F 2 "kbd_SW:CherryMX_Hotswap_2u" H 6050 5825 50  0001 C CNN
 F 3 "" H 6050 5825 50  0000 C CNN
 	1    6050 5825
@@
 F 0 "SW14" H 4100 6080 50  0000 C CNN
 F 1 "SW_PUSH" H 4100 5989 50  0000 C CNN
-F 2 "kbd_SW:CherryMX_Hotswap_1u" H 4100 5825 50  0001 C CNN
+F 2 "kbd_SW:CherryMX_Hotswap_1.25u" H 4100 5825 50  0001 C CNN
 F 3 "" H 4100 5825 50  0000 C CNN
 	1    4100 5825
@@
 F 0 "SW18" H 4750 6080 50  0000 C CNN
 F 1 "SW_PUSH" H 4750 5989 50  0000 C CNN
-F 2 "kbd_SW:CherryMX_Hotswap_1u" H 4750 5825 50  0001 C CNN
+F 2 "kbd_SW:CherryMX_Hotswap_2u" H 4750 5825 50  0001 C CNN
 F 3 "" H 4750 5825 50  0000 C CNN
 	1    4750 5825
@@
 F 0 "SW3" H 2800 3880 50  0000 C CNN
 F 1 "SW_PUSH" H 2800 3789 50  0000 C CNN
-F 2 "kbd_SW:CherryMX_Hotswap_1u" H 2800 3625 50  0001 C CNN
+F 2 "kbd_SW:CherryMX_Hotswap_1.5u" H 2800 3625 50  0001 C CNN
 F 3 "" H 2800 3625 50  0000 C CNN
 	1    2800 3625
@@
 F 0 "SW4" H 2800 4630 50  0000 C CNN
 F 1 "SW_PUSH" H 2800 4539 50  0000 C CNN
-F 2 "kbd_SW:CherryMX_Hotswap_1u" H 2800 4375 50  0001 C CNN
+F 2 "kbd_SW:CherryMX_Hotswap_1.75u" H 2800 4375 50  0001 C CNN
 F 3 "" H 2800 4375 50  0000 C CNN
 	1    2800 4375
@@
 F 0 "SW5" H 2800 5380 50  0000 C CNN
 F 1 "SW_PUSH" H 2800 5289 50  0000 C CNN
-F 2 "kbd_SW:CherryMX_Hotswap_1u" H 2800 5125 50  0001 C CNN
+F 2 "kbd_SW:CherryMX_Hotswap_2.25u" H 2800 5125 50  0001 C CNN
 F 3 "" H 2800 5125 50  0000 C CNN
 	1    2800 5125
@@
 F 0 "SW6" H 2800 6080 50  0000 C CNN
 F 1 "SW_PUSH" H 2800 5989 50  0000 C CNN
-F 2 "kbd_SW:CherryMX_Hotswap_1u" H 2800 5825 50  0001 C CNN
+F 2 "kbd_SW:CherryMX_Hotswap_1.25u" H 2800 5825 50  0001 C CNN
 F 3 "" H 2800 5825 50  0000 C CNN
 	1    2800 5825
@@
 F 0 "SW10" H 3450 6080 50  0000 C CNN
 F 1 "SW_PUSH" H 3450 5989 50  0000 C CNN
-F 2 "kbd_SW:CherryMX_Hotswap_1u" H 3450 5825 50  0001 C CNN
+F 2 "kbd_SW:CherryMX_Hotswap_1.25u" H 3450 5825 50  0001 C CNN
 F 3 "" H 3450 5825 50  0000 C CNN
 	1    3450 5825
@@
 	7100 7300 7600 7300
 NoConn ~ 7600 10900
-Connection ~ 6250 3925
 Connection ~ 6250 4675
 Connection ~ 6250 5425
@@
 	0    -1   -1   0
 $EndComp
-$Comp
-L Device:D D26
-U 1 1 612B3E34
-P 6900 3775
-F 0 "D26" V 6946 3696 50  0000 R CNN
-F 1 "D" V 6855 3696 50  0000 R CNN
-F 2 "kbd_Parts:Diode_SMD" H 6900 3775 50  0001 C CNN
-F 3 "~" H 6900 3775 50  0001 C CNN
-	1    6900 3775
-	0    -1   -1   0
-$EndComp
-Wire Wire Line
-	6900 3925 6250 3925
 Wire Wire Line
 	6900 4675 6250 4675
@@
 $EndComp
 Wire Wire Line
-	7550 3925 6900 3925
-Wire Wire Line
 	7550 4675 6900 4675
 Wire Wire Line
@@
 	12900 5335 13550 5335
 Wire Wire Line
-	10950 4585 11600 4585
-Connection ~ 10950 4585
-$Comp
-L Device:D D51
-U 1 1 60C8F1FE
-P 11600 4435
-F 0 "D51" V 11646 4356 50  0000 R CNN
-F 1 "D" V 11555 4356 50  0000 R CNN
-F 2 "kbd_Parts:Diode_SMD" H 11600 4435 50  0001 C CNN
-F 3 "~" H 11600 4435 50  0001 C CNN
-	1    11600 4435
-	0    1    1    0
-$EndComp
-Wire Wire Line
 	8400 4585 9000 4585
 Wire Wire Line
@@
 F 0 "SW51" H 11400 4540 50  0000 C CNN
 F 1 "SW_PUSH" H 11400 4449 50  0000 C CNN
-F 2 "kbd_SW:CherryMX_Hotswap_1u" H 11400 4285 50  0001 C CNN
+F 2 "kbd_SW:CherryMX_Hotswap_2.25u" H 11400 4285 50  0001 C CNN
 F 3 "" H 11400 4285 50  0000 C CNN
 	1    11400 4285
@@
 F 0 "SW48" H 10750 5290 50  0000 C CNN
 F 1 "SW_PUSH" H 10750 5199 50  0000 C CNN
-F 2 "kbd_SW:CherryMX_Hotswap_1u" H 10750 5035 50  0001 C CNN
+F 2 "kbd_SW:CherryMX_Hotswap_1.5u" H 10750 5035 50  0001 C CNN
 F 3 "" H 10750 5035 50  0000 C CNN
 	1    10750 5035
@@
 	1    0    0    -1
 $EndComp
+Connection ~ 6250 3925
+Wire Wire Line
+	7550 3925 6900 3925
+Wire Wire Line
+	6900 3925 6250 3925
+$Comp
+L Device:D D26
+U 1 1 612B3E34
+P 6900 3775
+F 0 "D26" V 6946 3696 50  0000 R CNN
+F 1 "D" V 6855 3696 50  0000 R CNN
+F 2 "kbd_Parts:Diode_SMD" H 6900 3775 50  0001 C CNN
+F 3 "~" H 6900 3775 50  0001 C CNN
+	1    6900 3775
+	0    -1   -1   0
+$EndComp
+Text GLabel 1700 7300 1    50   Input ~ 0
+LED
+Connection ~ 6900 3925
+Connection ~ 6900 5425
+Connection ~ 6900 6125
+Connection ~ 13550 4585
+Connection ~ 13550 5335
+Connection ~ 13550 6035
+Connection ~ 10950 4585
+$Comp
+L Device:D D51
+U 1 1 60C8F1FE
+P 11600 4435
+F 0 "D51" V 11646 4356 50  0000 R CNN
+F 1 "D" V 11555 4356 50  0000 R CNN
+F 2 "kbd_Parts:Diode_SMD" H 11600 4435 50  0001 C CNN
+F 3 "~" H 11600 4435 50  0001 C CNN
+	1    11600 4435
+	0    1    1    0
+$EndComp
+Wire Wire Line
+	10950 4585 11600 4585
+Wire Wire Line
+	11600 4585 12900 4585
+Connection ~ 11600 4585
+Connection ~ 12900 4585
+Wire Wire Line
+	11600 5335 12900 5335
+Connection ~ 11600 5335
+Connection ~ 12900 5335
 $EndSCHEMATC
